File: LCD.sch (KiCad schematic (older format))
At the start: 3 parts, among them P2 40pin_fpc_top_0_5mm

Commit message: Corrected FPC 40pin top 0.5mm connector, generated again gerber and ps files
Parts:
- C4, C5: symbol 100nF_0805 -> Capacitors_Smd0805:100nF_0805
- P2: symbol 40pin_fpc_top_0_5mm -> Fpc_Connectors:40pin_fpc_top_0_5mm
Changed lines of the file:
@@
-EESchema Schematic File Version 3
-LIBS:Capacitors_Smd0805
-LIBS:Capacitors_Smd_Tantal
-LIBS:Fpc_Connectors
-LIBS:Switching_Regulators
-LIBS:Diodes
-LIBS:Inductors
-LIBS:power
-LIBS:Resistors_Smd0603
-LIBS:Resistors_Smd0805
-LIBS:Symbols
-LIBS:Touch_Sensors
+EESchema Schematic File Version 4
 LIBS:TFT_LCD_4_3_AM480272H2T_V1_0-cache
 EELAYER 26 0
@@
 $EndDescr
 $Comp
-L GND #PWR047
+L power1:GND #PWR047
 U 1 1 578B809F
 P 1500 4950
@@
 LCD_VSYNC
 $Comp
-L GND #PWR049
+L power1:GND #PWR049
 U 1 1 578B83EB
 P 6050 2250
@@
 $EndComp
 $Comp
-L GND #PWR050
+L power1:GND #PWR050
 U 1 1 578B8405
 P 6050 2150
@@
 $EndComp
 $Comp
-L 3V3 #PWR051
+L power1:3V3 #PWR051
 U 1 1 57EC9FE0
 P 1650 2350
@@
 $EndComp
 $Comp
-L 3V3 #PWR052
+L power1:3V3 #PWR052
 U 1 1 57ECA1FC
 P 1650 2450
@@
 $EndComp
 $Comp
-L 100nF_0805 C5
+L Capacitors_Smd0805:100nF_0805 C5
 U 1 1 57FFFF60
 P 4650 2200
@@
 $EndComp
 $Comp
-L 100nF_0805 C4
+L Capacitors_Smd0805:100nF_0805 C4
 U 1 1 57FFFF8B
 P 2900 2200
@@
 $EndComp
 $Comp
-L GND #PWR053
+L power1:GND #PWR053
 U 1 1 580000DE
 P 2600 2200
@@
 	2700 2200 2600 2200
 $Comp
-L GND #PWR054
+L power1:GND #PWR054
 U 1 1 58000232
 P 4350 2200
@@
 	4450 2200 4350 2200
 $Comp
-L 40pin_fpc_top_0_5mm P2
+L Fpc_Connectors:40pin_fpc_top_0_5mm P2
 U 1 1 59F3ACC9
 P 6400 4100
